Commit message: Move ZED camera to chassis front and remove mast

File: fleet_description/urdf/amr.urdf.xacro (robot description, xacro)
@@ -51,7 +51,6 @@
   <!-- ZED camera (center of the camera body) -->
   <xacro:property name="zed_name"                value="zed"/>
-  <xacro:property name="zed_x"                   value="0.20"/>  <!-- in base_link -->
+  <xacro:property name="zed_x"                   value="0.268"/> <!-- in base_link: chassis front (0.25) + 2 mm band + zed_size_x/2 -->
   <xacro:property name="zed_y"                   value="0.0"/>
-  <xacro:property name="zed_height_above_chassis" value="0.20"/> <!-- camera center above top panel -->
   <xacro:property name="zed_baseline"            value="0.12"/>
   <xacro:property name="zed_mass"                value="0.124"/>
@@ -60,6 +59,4 @@
   <xacro:property name="zed_size_z"              value="0.030"/>
   <xacro:property name="zed_mesh_yaw"            value="0.0"/>   <!-- set to ${pi} if the mesh faces backwards -->
-  <xacro:property name="mast_size"               value="0.03"/>  <!-- square mast carrying the camera -->
-  <xacro:property name="mast_mass"               value="0.3"/>
   <!-- ====================== DERIVED VALUES ====================== -->
   <!-- base_link sits on the wheel axle; base_footprint is on the floor below it. -->
@@ -67,6 +64,5 @@
   <xacro:property name="chassis_top_z" value="${chassis_z + chassis_height / 2.0 + panel_thickness}"/>
   <xacro:property name="lidar_z"       value="${chassis_top_z + lidar_height_above_mount + lidar_scan_height}"/>
-  <xacro:property name="zed_z"         value="${chassis_top_z + zed_height_above_chassis}"/>
-  <xacro:property name="mast_length"   value="${zed_height_above_chassis - zed_size_z / 2.0}"/>
+  <xacro:property name="zed_z"         value="${chassis_z}"/>  <!-- camera centered on the front face of the chassis -->
   <!-- Mesh path: absolute file:// for Gazebo, package:// for RViz/URDF-only use. -->
   <xacro:if value="$(arg use_sim)">

File: fleet_description/urdf/amr_body.xacro (robot description, xacro)
@@ -1,4 +1,4 @@
 <?xml version="1.0"?>
-<!-- Chassis, top panel, accent band, camera mast, drive wheels and casters.
+<!-- Chassis, top panel, accent band, drive wheels and casters.
      base_footprint (floor) -> base_link (wheel-axle height, REP-105). -->
 <robot xmlns:xacro="http://www.ros.org/wiki/xacro">
@@ -108,24 +108,4 @@
       <origin xyz="0 0 ${chassis_z + chassis_height / 2.0 - stripe_drop - stripe_height / 2.0}" rpy="0 0 0"/>
     </joint>
-    <!-- Camera mast (accent color): panel top -> bottom of the camera -->
-    <link name="mast_link">
-      <visual>
-        <origin xyz="0 0 0" rpy="0 0 0"/>
-        <geometry><box size="${mast_size} ${mast_size} ${mast_length}"/></geometry>
-        <material name="accent"/>
-      </visual>
-      <collision>
-        <origin xyz="0 0 0" rpy="0 0 0"/>
-        <geometry><box size="${mast_size} ${mast_size} ${mast_length}"/></geometry>
-      </collision>
-      <xacro:box_inertial m="${mast_mass}" x="${mast_size}" y="${mast_size}" z="${mast_length}">
-        <origin xyz="0 0 0" rpy="0 0 0"/>
-      </xacro:box_inertial>
-    </link>
-    <joint name="mast_joint" type="fixed">
-      <parent link="base_link"/>
-      <child link="mast_link"/>
-      <origin xyz="${zed_x} ${zed_y} ${chassis_top_z + mast_length / 2.0}" rpy="0 0 0"/>
-    </joint>
     <!-- Drive wheels -->
     <xacro:wheel side="left"  y_sign="1.0"/>

File: fleet_description/urdf/gazebo.xacro (robot description, xacro)
@@ -40,5 +40,4 @@
     <xacro:gz_material link="top_panel_link"     rgba="${chassis_panel_rgba}" specular="0.4 0.4 0.4 1.0"/>
     <xacro:gz_material link="accent_stripe_link" rgba="${accent_rgba}"        specular="0.3 0.3 0.3 1.0"/>
-    <xacro:gz_material link="mast_link"          rgba="${accent_rgba}"        specular="0.3 0.3 0.3 1.0"/>
     <xacro:gz_material link="left_wheel_link"    rgba="${wheel_rgba}"         specular="0.05 0.05 0.05 1.0"/>
     <xacro:gz_material link="right_wheel_link"   rgba="${wheel_rgba}"         specular="0.05 0.05 0.05 1.0"/>
@@ -50,5 +49,4 @@
     <xacro:gz_keep_joint joint="top_panel_joint"/>
     <xacro:gz_keep_joint joint="accent_stripe_joint"/>
-    <xacro:gz_keep_joint joint="mast_joint"/>
     <xacro:gz_keep_joint joint="lidar_joint"/>
     <xacro:gz_keep_joint joint="caster_front_joint"/>
